File: HW/ibakey52.kicad_pcb (KiCad board)
At the start: 4 copper layers, 143.2 x 150.7 mm, 107 parts, among them J1 AudioJack4, SW1 GATERON-MX-HOTSWAP-RGB, SW10 GATERON-MX-HOTSWAP-RGB, SW11 GATERON-MX-HOTSWAP-RGB, SW12 GATERON-MX-HOTSWAP-RGB, SW13 GATERON-MX-HOTSWAP-RGB, SW14 GATERON-MX-HOTSWAP-RGB, SW15 GATERON-MX-HOTSWAP-RGB, SW16 GATERON-MX-HOTSWAP-RGB, SW17 GATERON-MX-HOTSWAP-RGB, SW18 GATERON-MX-HOTSWAP-RGB, SW19 GATERON-MX-HOTSWAP-RGB, SW2 GATERON-MX-HOTSWAP-RGB, SW20 GATERON-MX-HOTSWAP-RGB, SW21 GATERON-MX-HOTSWAP-RGB, SW22 GATERON-MX-HOTSWAP-RGB, SW23 GATERON-MX-HOTSWAP-RGB, SW24 GATERON-MX-HOTSWAP-RGB, SW25 GATERON-MX-HOTSWAP-RGB, SW26 GATERON-MX-HOTSWAP-RGB, SW3 GATERON-MX-HOTSWAP-RGB, SW4 GATERON-MX-HOTSWAP-RGB, SW5 GATERON-MX-HOTSWAP-RGB, SW6 GATERON-MX-HOTSWAP-RGB, SW7 GATERON-MX-HOTSWAP-RGB, SW8 GATERON-MX-HOTSWAP-RGB, SW9 GATERON-MX-HOTSWAP-RGB, U1 Nice!Nano

Commit message: Renaming project
Parts:
- added JP1: SolderJumper_2_Open, Jumper:SolderJumper-2_P1.3mm_Open_TrianglePad1.0x1.5mm, F.Cu at (218.7, 21.3)
- added JP10: SolderJumper_2_Open, Jumper:SolderJumper-2_P1.3mm_Open_TrianglePad1.0x1.5mm, F.Cu at (223.0, 21.3)
- added JP11: SolderJumper_2_Open, Jumper:SolderJumper-2_P1.3mm_Open_TrianglePad1.0x1.5mm, F.Cu at (223.0, 24.8)
- added JP12: SolderJumper_2_Open, Jumper:SolderJumper-2_P1.3mm_Open_TrianglePad1.0x1.5mm, F.Cu at (223.0, 28.4)
- added JP13: SolderJumper_2_Open, Jumper:SolderJumper-2_P1.3mm_Open_TrianglePad1.0x1.5mm, F.Cu at (223.0, 31.9)
- added JP14: SolderJumper_2_Open, Jumper:SolderJumper-2_P1.3mm_Open_TrianglePad1.0x1.5mm, F.Cu at (223.0, 35.5)
- added JP15: SolderJumper_2_Open, Jumper:SolderJumper-2_P1.3mm_Open_TrianglePad1.0x1.5mm, F.Cu at (223.0, 39.0)
- added JP16: SolderJumper_2_Open, Jumper:SolderJumper-2_P1.3mm_Open_TrianglePad1.0x1.5mm, F.Cu at (223.0, 42.6)
- added JP17: SolderJumper_2_Open, Jumper:SolderJumper-2_P1.3mm_Open_TrianglePad1.0x1.5mm, F.Cu at (223.0, 46.1)
- added JP18: SolderJumper_2_Open, Jumper:SolderJumper-2_P1.3mm_Open_TrianglePad1.0x1.5mm, F.Cu at (223.0, 49.7)
- added JP19: SolderJumper_2_Open, Jumper:SolderJumper-2_P1.3mm_Open_TrianglePad1.0x1.5mm, F.Cu at (227.4, 21.3)
- added JP2: SolderJumper_2_Open, Jumper:SolderJumper-2_P1.3mm_Open_TrianglePad1.0x1.5mm, F.Cu at (218.7, 24.8)
- added JP20: SolderJumper_2_Open, Jumper:SolderJumper-2_P1.3mm_Open_TrianglePad1.0x1.5mm, F.Cu at (227.4, 24.8)
- added JP21: SolderJumper_2_Open, Jumper:SolderJumper-2_P1.3mm_Open_TrianglePad1.0x1.5mm, F.Cu at (227.4, 28.4)
- added JP22: SolderJumper_2_Open, Jumper:SolderJumper-2_P1.3mm_Open_TrianglePad1.0x1.5mm, F.Cu at (227.4, 31.9)
- added JP23: SolderJumper_2_Open, Jumper:SolderJumper-2_P1.3mm_Open_TrianglePad1.0x1.5mm, F.Cu at (227.4, 35.5)
- added JP24: SolderJumper_2_Open, Jumper:SolderJumper-2_P1.3mm_Open_TrianglePad1.0x1.5mm, F.Cu at (227.4, 39.0)
- added JP25: SolderJumper_2_Open, Jumper:SolderJumper-2_P1.3mm_Open_TrianglePad1.0x1.5mm, F.Cu at (227.4, 42.6)
- added JP26: SolderJumper_2_Open, Jumper:SolderJumper-2_P1.3mm_Open_TrianglePad1.0x1.5mm, F.Cu at (227.4, 46.1)
- added JP27: SolderJumper_2_Open, Jumper:SolderJumper-2_P1.3mm_Open_TrianglePad1.0x1.5mm, F.Cu at (227.4, 49.7)
- added JP28: SolderJumper_2_Open, Jumper:SolderJumper-2_P1.3mm_Open_TrianglePad1.0x1.5mm, F.Cu at (231.7, 21.3)
- added JP29: SolderJumper_2_Open, Jumper:SolderJumper-2_P1.3mm_Open_TrianglePad1.0x1.5mm, F.Cu at (231.7, 24.8)
- added JP3: SolderJumper_2_Open, Jumper:SolderJumper-2_P1.3mm_Open_TrianglePad1.0x1.5mm, F.Cu at (218.7, 28.4)
- added JP30: SolderJumper_2_Open, Jumper:SolderJumper-2_P1.3mm_Open_TrianglePad1.0x1.5mm, F.Cu at (231.7, 28.4)
- added JP31: SolderJumper_2_Open, Jumper:SolderJumper-2_P1.3mm_Open_TrianglePad1.0x1.5mm, F.Cu at (231.7, 31.9)
- added JP32: SolderJumper_2_Open, Jumper:SolderJumper-2_P1.3mm_Open_TrianglePad1.0x1.5mm, F.Cu at (231.7, 35.5)
- added JP33: SolderJumper_2_Open, Jumper:SolderJumper-2_P1.3mm_Open_TrianglePad1.0x1.5mm, F.Cu at (231.7, 39.0)
- added JP34: SolderJumper_2_Open, Jumper:SolderJumper-2_P1.3mm_Open_TrianglePad1.0x1.5mm, F.Cu at (231.7, 42.6)
- added JP35: SolderJumper_2_Open, Jumper:SolderJumper-2_P1.3mm_Open_TrianglePad1.0x1.5mm, F.Cu at (231.7, 46.1)
- added JP36: SolderJumper_2_Open, Jumper:SolderJumper-2_P1.3mm_Open_TrianglePad1.0x1.5mm, F.Cu at (231.7, 49.7)
- added JP37: SolderJumper_2_Open, Jumper:SolderJumper-2_P1.3mm_Open_TrianglePad1.0x1.5mm, F.Cu at (236.1, 21.3)
- added JP38: SolderJumper_2_Open, Jumper:SolderJumper-2_P1.3mm_Open_TrianglePad1.0x1.5mm, F.Cu at (236.1, 24.8)
- added JP39: SolderJumper_2_Open, Jumper:SolderJumper-2_P1.3mm_Open_TrianglePad1.0x1.5mm, F.Cu at (236.1, 28.4)
- added JP4: SolderJumper_2_Open, Jumper:SolderJumper-2_P1.3mm_Open_TrianglePad1.0x1.5mm, F.Cu at (177.1, 41.5)
- added JP40: SolderJumper_2_Open, Jumper:SolderJumper-2_P1.3mm_Open_TrianglePad1.0x1.5mm, F.Cu at (236.1, 31.9)
- added JP41: SolderJumper_2_Open, Jumper:SolderJumper-2_P1.3mm_Open_TrianglePad1.0x1.5mm, F.Cu at (236.1, 35.5)
- added JP42: SolderJumper_2_Open, Jumper:SolderJumper-2_P1.3mm_Open_TrianglePad1.0x1.5mm, F.Cu at (236.1, 39.0)
- added JP43: SolderJumper_2_Open, Jumper:SolderJumper-2_P1.3mm_Open_TrianglePad1.0x1.5mm, F.Cu at (236.1, 42.6)
- added JP44: SolderJumper_2_Open, Jumper:SolderJumper-2_P1.3mm_Open_TrianglePad1.0x1.5mm, F.Cu at (236.1, 46.1)
- added JP45: SolderJumper_2_Open, Jumper:SolderJumper-2_P1.3mm_Open_TrianglePad1.0x1.5mm, F.Cu at (236.1, 49.7)
- added JP46: SolderJumper_2_Open, Jumper:SolderJumper-2_P1.3mm_Open_TrianglePad1.0x1.5mm, F.Cu at (240.4, 21.3)
- added JP47: SolderJumper_2_Open, Jumper:SolderJumper-2_P1.3mm_Open_TrianglePad1.0x1.5mm, F.Cu at (240.4, 24.8)
- added JP48: SolderJumper_2_Open, Jumper:SolderJumper-2_P1.3mm_Open_TrianglePad1.0x1.5mm, F.Cu at (240.4, 28.4)
- added JP49: SolderJumper_2_Open, Jumper:SolderJumper-2_P1.3mm_Open_TrianglePad1.0x1.5mm, F.Cu at (240.4, 31.9)
- added JP5: SolderJumper_2_Open, Jumper:SolderJumper-2_P1.3mm_Open_TrianglePad1.0x1.5mm, F.Cu at (218.7, 35.5)
- added JP50: SolderJumper_2_Open, Jumper:SolderJumper-2_P1.3mm_Open_TrianglePad1.0x1.5mm, F.Cu at (240.4, 35.5)
- added JP51: SolderJumper_2_Open, Jumper:SolderJumper-2_P1.3mm_Open_TrianglePad1.0x1.5mm, F.Cu at (240.4, 39.0)
- added JP52: SolderJumper_2_Open, Jumper:SolderJumper-2_P1.3mm_Open_TrianglePad1.0x1.5mm, F.Cu at (240.4, 42.6)
- added JP6: SolderJumper_2_Open, Jumper:SolderJumper-2_P1.3mm_Open_TrianglePad1.0x1.5mm, F.Cu at (218.7, 39.0)
- added JP7: SolderJumper_2_Open, Jumper:SolderJumper-2_P1.3mm_Open_TrianglePad1.0x1.5mm, F.Cu at (218.7, 42.6)
- added JP8: SolderJumper_2_Open, Jumper:SolderJumper-2_P1.3mm_Open_TrianglePad1.0x1.5mm, F.Cu at (218.7, 46.1)
- added JP9: SolderJumper_2_Open, Jumper:SolderJumper-2_P1.3mm_Open_TrianglePad1.0x1.5mm, F.Cu at (218.7, 49.7)
Connections:
- U1 pad 1: GND -> /PIN1
- U1 pad 10: unconnected-(U1-D6/P1.00-Pad10) -> /PIN10
- U1 pad 11: unconnected-(U1-D7/P0.11-Pad11) -> /PIN11
- U1 pad 12: unconnected-(U1-D8/P1.04-Pad12) -> /PIN12
- U1 pad 13: unconnected-(U1-D9/P1.06-Pad13) -> /PIN13
- U1 pad 14: unconnected-(U1-D10/P0.09-Pad14) -> /PIN14
- U1 pad 15: unconnected-(U1-D16/P0.10-Pad15) -> /PIN15
- U1 pad 16: unconnected-(U1-D14/P1.11-Pad16) -> /PIN16
- U1 pad 17: unconnected-(U1-D15/P1.13-Pad17) -> /PIN17
- U1 pad 18: unconnected-(U1-D18/P1.15-Pad18) -> /PIN18
- U1 pad 19: unconnected-(U1-D19/P0.02-Pad19) -> /PIN19
- U1 pad 2: unconnected-(U1-D1/P0.06-Pad2) -> /PIN2
- U1 pad 20: unconnected-(U1-D20/P0.29-Pad20) -> /PIN20
- U1 pad 21: unconnected-(U1-D21/P0.31-Pad21) -> /PIN21
- U1 pad 22: unconnected-(U1-3.3V-Pad22) -> /PIN22
- U1 pad 23: unconnected-(U1-~{RST}-Pad23) -> /PIN23
- U1 pad 24: GND -> /PIN24
- U1 pad 25: unconnected-(U1-VBATT-Pad25) -> /PIN25
- U1 pad 26: unconnected-(U1-VBATT-Pad26) -> /PIN26
- U1 pad 3: unconnected-(U1-D0/P0.08-Pad3) -> /PIN3
- U1 pad 4: GND -> /PIN4
- U1 pad 5: GND -> /PIN5
- U1 pad 6: unconnected-(U1-D2/P0.17-Pad6) -> /PIN6
- U1 pad 7: unconnected-(U1-D3/P0.20-Pad7) -> /PIN7
- U1 pad 8: unconnected-(U1-D4/P0.22-Pad8) -> /PIN8
- U1 pad 9: unconnected-(U1-D5/P0.24-Pad9) -> /PIN9

Commit message: matrix routed
Parts:
- added D27: D1213A-02WLQ-7, Package_TO_SOT_SMD:SOT-323_SC-70, F.Cu at (135.0, 36.1)
- added D28: DESD5V0U1BA-7, Diode_SMD:D_SOD-323, F.Cu at (148.5, 32.5)
- added D29: DESD5V0U1BA-7, Diode_SMD:D_SOD-323, F.Cu at (98.4, 45.3)
- added D30: DESD5V0U1BA-7, Diode_SMD:D_SOD-323, B.Cu at (91.0, 41.2)
- added D31: DESD5V0U1BA-7, Diode_SMD:D_SOD-323, B.Cu at (98.4, 45.3)
- added J2: USB_C_Receptacle_USB2.0_16P, CONN-USB:GCT_USB4520-03-0-A_REVA, B.Cu at (135.0, 27.8)
- added J3: USB_C_Receptacle_USB2.0_16P, CONN-USB:GCT_USB4520-03-0-A_REVA, F.Cu at (135.0, 27.8)
- added J4: ~, Connector_JST:JST_PH_S2B-PH-K_1x02_P2.00mm_Horizontal, F.Cu at (160.5, 37.6)
- added JP53: SolderJumper_2_Open, JUMPER:SJMP1.3mm, F.Cu at (87.5, 29.2)
- added JP54: SolderJumper_2_Open, JUMPER:SJMP1.3mm, B.Cu at (87.5, 39.4)
- added JP55: SolderJumper_2_Open, JUMPER:SJMP1.3mm, F.Cu at (87.5, 31.8)
- added JP56: SolderJumper_2_Open, JUMPER:SJMP1.3mm, B.Cu at (87.5, 36.8)
- added JP57: SolderJumper_2_Open, JUMPER:SJMP1.3mm, F.Cu at (87.5, 36.8)
- added JP58: SolderJumper_2_Open, JUMPER:SJMP1.3mm, B.Cu at (87.5, 31.8)
- added JP59: SolderJumper_2_Open, JUMPER:SJMP1.3mm, F.Cu at (87.5, 39.4)
- added JP60: SolderJumper_2_Open, JUMPER:SJMP1.3mm, B.Cu at (87.5, 29.2)
- added JP61: SolderJumper_2_Open, JUMPER:SJMP1.3mm, F.Cu at (100.9, 47.6)
- added JP62: SolderJumper_2_Open, JUMPER:SJMP1.3mm, B.Cu at (100.9, 43.0)
- added JP63: SolderJumper_2_Open, JUMPER:SJMP1.3mm, F.Cu at (100.9, 43.0)
- added JP64: SolderJumper_2_Open, JUMPER:SJMP1.3mm, B.Cu at (100.9, 47.6)
- added L1: DLW21HN900SQ2L, IND-SMD-CHOKE:FIL_DLW21HN900SQ2L, F.Cu at (139.5, 36.5)
- added LF1: MPZ1608S601ATA00, Inductor_SMD:L_0603_1608Metric, F.Cu at (139.5, 34.7)
- added LF2: MPZ1608S601ATA00, Inductor_SMD:L_0603_1608Metric, F.Cu at (98.2, 47.6)
- added LF3: MPZ1608S601ATA00, Inductor_SMD:L_0603_1608Metric, F.Cu at (91.0, 41.2)
- added LF4: MPZ1608S601ATA00, Inductor_SMD:L_0603_1608Metric, F.Cu at (98.2, 43.0)
- added LF5: MPZ1608S601ATA00, Inductor_SMD:L_0603_1608Metric, F.Cu at (148.5, 36.0)
- added Q1: Si2371EDS, Package_TO_SOT_SMD:SOT-23, F.Cu at (156.7, 36.6)
- added R1: r=2.2k, Resistor_SMD:R_0603_1608Metric, F.Cu at (131.9, 35.0)
- added R2: r=2.2k, Resistor_SMD:R_0603_1608Metric, F.Cu at (131.9, 36.5)
- added R3: r=100k, Resistor_SMD:R_0603_1608Metric, F.Cu at (156.3, 33.9)
- added SW27: SSSS811101, SWITCH-SMD-SLIDE:SSSS811101, F.Cu at (162.9, 27.7)
- added SW28: SSSS811101, SWITCH-SMD-SLIDE:SSSS811101, B.Cu at (162.9, 27.7)
- added SW29: SW_Push, SWITCH-SMD-PB:EVQ-PUL02K, F.Cu at (154.0, 28.2)
- JP1, JP10, JP11, JP12, JP13, JP2, JP27, JP28, JP29, JP3, JP30, JP31, JP32, JP33, JP34, JP35, JP36, JP37, JP38, JP39, JP4, JP5, JP6, JP7, JP8, JP9: footprint Jumper:SolderJumper-2_P1.3mm_Open_TrianglePad1.0x1.5mm -> JUMPER:SJMP1.3mm
- JP14, JP15, JP16, JP17, JP18, JP19, JP20, JP21, JP22, JP23, JP24, JP25, JP26, JP40, JP41, JP42, JP43, JP44, JP45, JP46, JP47, JP48, JP49, JP50, JP51, JP52: footprint Jumper:SolderJumper-2_P1.3mm_Open_TrianglePad1.0x1.5mm -> JUMPER:SJMP1.3mm; moved to B.Cu
- moved JP52 70.9 mm to (169.5, 42.0), turned to 90 degrees
- moved JP51 68.4 mm to (172.0, 42.0), turned to 90 degrees
- moved JP50 66.2 mm to (174.6, 42.0), turned to 90 degrees
- moved JP49 64.1 mm to (177.1, 42.0), turned to 90 degrees
- moved JP48 62.3 mm to (179.6, 42.0), turned to 90 degrees
- moved JP27 60.7 mm to (169.5, 31.2), turned to -90 degrees
- moved JP47 60.7 mm to (182.2, 42.0), turned to 90 degrees
- moved JP28 60.5 mm to (172.0, 31.2), turned to -90 degrees
- moved JP26 59.8 mm to (169.5, 31.2), turned to -90 degrees
- moved JP46 59.4 mm to (184.7, 42.0), turned to 90 degrees
- moved JP29 57.5 mm to (174.6, 31.2), turned to -90 degrees
- moved JP25 56.5 mm to (172.0, 31.2), turned to -90 degrees
- moved JP30 54.7 mm to (177.1, 31.2), turned to -90 degrees
- moved JP24 53.4 mm to (174.6, 31.2), turned to -90 degrees
- moved JP1 53.4 mm to (169.5, 42.0), turned to 90 degrees
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Connections:
- Display1 pad 1: unconnected-(Display1-MOSI-Pad1) -> Net-(Display1-MOSI)
- Display1 pad 2: unconnected-(Display1-SCK-Pad2) -> Net-(Display1-SCK)
- Display1 pad 3: unconnected-(Display1-VCC-Pad3) -> +3.3V
- Display1 pad 4: unconnected-(Display1-GND-Pad4) -> Net-(Display1-GND)
- Display1 pad 5: unconnected-(Display1-CS-Pad5) -> Net-(Display1-CS)
- J1 pad R1: unconnected-(J1-PadR1) -> Net-(D30-A2)
- J1 pad R2: unconnected-(J1-PadR2) -> GND
- J1 pad S: unconnected-(J1-PadS) -> Net-(D29-A2)
- J1 pad T: unconnected-(J1-PadT) -> Net-(D31-A2)
- JP1 pad 1: unconnected-(JP1-A-Pad1) -> /PIN1
- JP1 pad 2: /PIN1 -> GND
- JP10 pad 1: unconnected-(JP10-A-Pad1) -> /PIN10
- JP10 pad 2: /PIN10 -> /ROW0
- JP11 pad 1: unconnected-(JP11-A-Pad1) -> /PIN11
- JP11 pad 2: /PIN11 -> /ROW1
- JP12 pad 1: unconnected-(JP12-A-Pad1) -> /PIN12
- JP12 pad 2: /PIN12 -> /ROW2
- JP13 pad 1: unconnected-(JP13-A-Pad1) -> /PIN13
- JP13 pad 2: /PIN13 -> /ROW3
- JP14 pad 1: unconnected-(JP14-A-Pad1) -> /PIN14
- JP14 pad 2: /PIN14 -> /ROW3
- JP15 pad 1: unconnected-(JP15-A-Pad1) -> /PIN15
- JP15 pad 2: /PIN15 -> /ROW2
- JP16 pad 1: unconnected-(JP16-A-Pad1) -> /PIN16
- JP16 pad 2: /PIN16 -> /ROW1
- JP17 pad 1: unconnected-(JP17-A-Pad1) -> /PIN17
- JP17 pad 2: /PIN17 -> /ROW0
- JP18 pad 1: unconnected-(JP18-A-Pad1) -> /PIN18
- JP18 pad 2: /PIN18 -> /LED_D
- JP19 pad 1: unconnected-(JP19-A-Pad1) -> /PIN19
- JP19 pad 2: /PIN19 -> /CS
- JP2 pad 1: unconnected-(JP2-A-Pad1) -> /PIN2
- JP2 pad 2: /PIN2 -> /SDA
- JP20 pad 1: unconnected-(JP20-A-Pad1) -> /PIN20
- JP20 pad 2: /PIN20 -> /MOSI
- JP21 pad 1: unconnected-(JP21-A-Pad1) -> /PIN21
- JP21 pad 2: /PIN21 -> /SCK
- JP22 pad 1: unconnected-(JP22-A-Pad1) -> /PIN22
- JP22 pad 2: /PIN22 -> GND
- JP23 pad 1: unconnected-(JP23-A-Pad1) -> /PIN23
- JP23 pad 2: /PIN23 -> GND
- JP24 pad 1: unconnected-(JP24-A-Pad1) -> /PIN24
- JP24 pad 2: /PIN24 -> /SCL
- JP25 pad 1: unconnected-(JP25-A-Pad1) -> /PIN25
- JP25 pad 2: /PIN25 -> /SDA
- JP26 pad 1: unconnected-(JP26-A-Pad1) -> /PIN26
- JP26 pad 2: /PIN26 -> GND
- JP27 pad 1: unconnected-(JP27-A-Pad1) -> /PIN26
- JP27 pad 2: /PIN26 -> VBATT
- JP28 pad 1: unconnected-(JP28-A-Pad1) -> /PIN25
- JP28 pad 2: /PIN25 -> VBATT
- JP29 pad 1: unconnected-(JP29-A-Pad1) -> /PIN24
- JP29 pad 2: /PIN24 -> GND
- JP3 pad 1: unconnected-(JP3-A-Pad1) -> /PIN3
- JP3 pad 2: /PIN3 -> /SCL
- JP30 pad 1: unconnected-(JP30-A-Pad1) -> /PIN23
- JP30 pad 2: /PIN23 -> /~{RST}
- JP31 pad 1: unconnected-(JP31-A-Pad1) -> /PIN22
- JP31 pad 2: /PIN22 -> +3.3V
- JP32 pad 1: unconnected-(JP32-A-Pad1) -> /PIN21
- JP32 pad 2: /PIN21 -> unconnected-(JP32-B-Pad2)
- JP33 pad 1: unconnected-(JP33-A-Pad1) -> /PIN20
- JP33 pad 2: /PIN20 -> /COL0
- JP34 pad 1: unconnected-(JP34-A-Pad1) -> /PIN19
- JP34 pad 2: /PIN19 -> /COL1
- JP35 pad 1: unconnected-(JP35-A-Pad1) -> /PIN18
- JP35 pad 2: /PIN18 -> /COL2
- JP36 pad 1: unconnected-(JP36-A-Pad1) -> /PIN17
- JP36 pad 2: /PIN17 -> /COL3
- JP37 pad 1: unconnected-(JP37-A-Pad1) -> /PIN16
- JP37 pad 2: /PIN16 -> /COL4
- JP38 pad 1: unconnected-(JP38-A-Pad1) -> /PIN15
- JP38 pad 2: /PIN15 -> /COL5
- JP39 pad 1: unconnected-(JP39-A-Pad1) -> /PIN14
- JP39 pad 2: /PIN14 -> /ROW4
- JP4 pad 1: unconnected-(JP4-A-Pad1) -> /PIN4
- JP4 pad 2: /PIN4 -> GND
- JP40 pad 1: unconnected-(JP40-A-Pad1) -> /PIN13
- JP40 pad 2: /PIN13 -> /ROW4
- JP41 pad 1: unconnected-(JP41-A-Pad1) -> /PIN12
- JP41 pad 2: /PIN12 -> /COL5
- JP42 pad 1: unconnected-(JP42-A-Pad1) -> /PIN11
- JP42 pad 2: /PIN11 -> /COL4
- JP43 pad 1: unconnected-(JP43-A-Pad1) -> /PIN10
- JP43 pad 2: /PIN10 -> /COL3
- JP44 pad 1: unconnected-(JP44-A-Pad1) -> /PIN9
- JP44 pad 2: /PIN9 -> /COL2
- JP45 pad 1: unconnected-(JP45-A-Pad1) -> /PIN8
- JP45 pad 2: /PIN8 -> /COL1
- JP46 pad 1: unconnected-(JP46-A-Pad1) -> /PIN7
- JP46 pad 2: /PIN7 -> /COL0
- JP47 pad 1: unconnected-(JP47-A-Pad1) -> /PIN6
- JP47 pad 2: /PIN6 -> unconnected-(JP47-B-Pad2)
- JP48 pad 1: unconnected-(JP48-A-Pad1) -> /PIN5
- JP48 pad 2: /PIN5 -> +3.3V
- JP49 pad 1: unconnected-(JP49-A-Pad1) -> /PIN4
- JP49 pad 2: /PIN4 -> /~{RST}
- JP5 pad 1: unconnected-(JP5-A-Pad1) -> /PIN5
- JP5 pad 2: /PIN5 -> GND
- JP50 pad 1: unconnected-(JP50-A-Pad1) -> /PIN3
- JP50 pad 2: /PIN3 -> GND
- JP51 pad 1: unconnected-(JP51-A-Pad1) -> /PIN2
- JP51 pad 2: /PIN2 -> VBATT
- JP52 pad 1: unconnected-(JP52-A-Pad1) -> /PIN1
- JP52 pad 2: /PIN1 -> VBATT
- JP6 pad 1: unconnected-(JP6-A-Pad1) -> /PIN6
- JP6 pad 2: /PIN6 -> /SCK
- JP7 pad 1: unconnected-(JP7-A-Pad1) -> /PIN7
- JP7 pad 2: /PIN7 -> /MOSI
- JP8 pad 1: unconnected-(JP8-A-Pad1) -> /PIN8
- JP8 pad 2: /PIN8 -> /CS
- JP9 pad 1: unconnected-(JP9-A-Pad1) -> /PIN9
- JP9 pad 2: /PIN9 -> /LED_D
Routing:
- net /ROW4: track 0.00 -> 245.2 mm, vias 0 -> 2
- net Net-(SW24-DOUT): track 0.00 -> 190.4 mm, vias 0 -> 2
- net /COL0: track 58.5 -> 234.2 mm, vias 0 -> 6
- net /ROW3: track 110.9 -> 279.2 mm, vias 6 -> 8
- net Net-(SW12-DOUT): track 0.00 -> 156.6 mm, vias 1 -> 2
- net Net-(SW6-DOUT): track 0.00 -> 156.6 mm, vias 1 -> 2
- net Net-(SW18-DOUT): track 3.56 -> 156.6 mm
- net /COL1: track 58.5 -> 202.2 mm, vias 0 -> 6
- net /MOSI: track 0.00 -> 130.3 mm, vias 0 -> 3
- net /ROW2: track 111.7 -> 238.7 mm, vias 6 -> 8
- net /CS: track 0.00 -> 126.5 mm, vias 0 -> 3
- net /LED_D: track 0.00 -> 121.4 mm, vias 1 -> 3
- net /SCK: track 0.00 -> 112.8 mm, vias 0 -> 2
- net /COL4: track 0.00 -> 109.8 mm, vias 0 -> 4
- net +3.3V: track 0.00 -> 108.7 mm, vias 0 -> 2
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- added copper zone on B.Cu, net GND
- added copper zone on In1.Cu, net GND
- added copper zone on B.Cu, net Net-(D27-common)
- added copper zone on F.Cu, net Net-(D27-common)
- added copper zone on In1.Cu, net Net-(D27-common)
- added copper zone on In2.Cu, net Net-(D27-common)
- added copper zone on F.Cu, net VDD
- added copper zone on In2.Cu, net VDD

Commit message: correcting switch footprint & updating LED routing
Parts:
- removed JP1, JP26, JP27, JP52: SolderJumper_2_Open, JUMPER:SJMP1.3mm
- R3: value r=100k -> r=2.2k
- moved C10 5.49 mm to (154.8, 71.3), turned to 180 degrees
- moved C11 5.49 mm to (174.3, 75.0), turned to 180 degrees
- moved C12 5.49 mm to (193.8, 75.0), turned to 180 degrees
- moved C15 5.49 mm to (135.3, 87.3), turned to 180 degrees
- moved C16 5.49 mm to (154.8, 90.8), turned to 180 degrees
- moved C17 5.49 mm to (174.3, 94.5), turned to 180 degrees
- moved C18 5.49 mm to (193.8, 94.5), turned to 180 degrees
- moved C21 5.49 mm to (135.3, 106.8), turned to 180 degrees
- moved C22 5.49 mm to (154.8, 110.3), turned to 180 degrees
- moved C23 5.49 mm to (174.3, 114.0), turned to 180 degrees
- moved C24 5.49 mm to (193.8, 114.0), turned to 180 degrees
- moved C3 5.49 mm to (135.3, 48.3), turned to 180 degrees
- moved C4 5.49 mm to (154.8, 51.8), turned to 180 degrees
- moved C5 5.49 mm to (174.3, 55.5), turned to 180 degrees
- moved C6 5.49 mm to (193.8, 55.5), turned to 180 degrees
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Connections:
- J2 pad A6: (no net) -> /USB_D+
- J2 pad A7: (no net) -> /USB_D-
- J3 pad A1: Net-(D27-common) -> Net-(J3-GND-PadA1)
- J3 pad A4: Net-(D28-A2) -> Net-(J3-VBUS-PadA4)
- J3 pad A5: Net-(J2-CC1) -> unconnected-(J3-CC1-PadA5)
- J3 pad A6: /USB_D+ -> unconnected-(J3-D+-PadA6)
- J3 pad A7: /USB_D- -> unconnected-(J3-D--PadA7)
- J3 pad A8: unconnected-(J2-SBU1-PadA8) -> unconnected-(J3-SBU1-PadA8)
- J3 pad B1: Net-(D27-common) -> Net-(J3-GND-PadA1)
- J3 pad B4: Net-(D28-A2) -> Net-(J3-VBUS-PadA4)
- J3 pad B5: Net-(J2-CC2) -> unconnected-(J3-CC2-PadB5)
- J3 pad B6: (no net) -> unconnected-(J3-D+-PadB6)
- J3 pad B7: (no net) -> unconnected-(J3-D--PadB7)
- J3 pad B8: unconnected-(J2-SBU2-PadB8) -> unconnected-(J3-SBU2-PadB8)
- J3 pad S1: unconnected-(J2-SHIELD-PadS1) -> unconnected-(J3-SHIELD-PadS1)
- Q1 pad 1: VBUS -> Net-(Q1-G)
- R3 pad 1: VBUS -> Net-(Q2-G)
- R3 pad 2: GND -> VBUS
- U1 pad 1: /PIN1 -> /PIN2
- U1 pad 10: /PIN10 -> /PIN11
- U1 pad 11: /PIN11 -> /PIN12
- U1 pad 12: /PIN12 -> /PIN13
- U1 pad 13: /PIN13 -> /PIN14
- U1 pad 14: /PIN14 -> /PIN15
- U1 pad 15: /PIN15 -> /PIN16
- U1 pad 16: /PIN16 -> /PIN17
- U1 pad 17: /PIN17 -> /PIN18
- U1 pad 18: /PIN18 -> /PIN19
- U1 pad 19: /PIN19 -> /PIN20
- U1 pad 2: /PIN2 -> /PIN3
- U1 pad 20: /PIN20 -> /PIN21
- U1 pad 21: /PIN21 -> /PIN22
- U1 pad 22: /PIN22 -> /PIN23
- U1 pad 23: /PIN23 -> /PIN24
- U1 pad 24: /PIN24 -> /PIN25
- U1 pad 3: /PIN3 -> /PIN4
- U1 pad 4: /PIN4 -> /PIN5
- U1 pad 5: /PIN5 -> /PIN6
- U1 pad 6: /PIN6 -> /PIN7
- U1 pad 7: /PIN7 -> /PIN8
- U1 pad 8: /PIN8 -> /PIN9
- U1 pad 9: /PIN9 -> /PIN10
Routing:
- net GND: track 14.1 -> 204.2 mm, vias 51 -> 63
- net Net-(SW1-DOUT): track 24.7 -> 42.4 mm
- net Net-(SW7-DOUT): track 24.7 -> 42.4 mm
- net Net-(SW13-DOUT): track 24.7 -> 42.4 mm
- net Net-(SW25-DOUT): track 25.0 -> 41.2 mm
- net Net-(SW18-DOUT): track 156.6 -> 171.0 mm
- net Net-(SW12-DOUT): track 156.6 -> 171.0 mm
- net Net-(SW6-DOUT): track 156.6 -> 171.0 mm
- net Net-(SW2-DOUT): track 24.0 -> 36.7 mm
- net Net-(SW8-DOUT): track 24.0 -> 36.7 mm
- net Net-(SW20-DOUT): track 24.0 -> 36.7 mm
- net Net-(SW14-DOUT): track 24.0 -> 36.7 mm
- net Net-(SW19-DOUT): track 24.7 -> 37.2 mm
- net Net-(SW5-DOUT): track 26.2 -> 38.0 mm
- net Net-(SW23-DOUT): track 26.2 -> 38.0 mm
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